File: KiCad/OPA990 Breakout.kicad_pcb (KiCad board)
At the start: 4 copper layers, 21.6 x 12.7 mm, 15 parts, among them J1 Conn_01x03, J2 Conn_01x03, U1 OPA99X

Commit message: updated kicad files
Parts:
- added REF**: Icon_Small, Fried_Electronics_Footprints:Icon_Small, B.Cu at (144.8, 99.7)
- added kibuzzard-659D8DDF: G***, kibuzzard-659D8DDF, B.Cu at (145.8, 93.3)
- added kibuzzard-659D8E26: G***, kibuzzard-659D8E26, B.Cu at (146.4, 92.1)
- added kibuzzard-659D8E62: G***, kibuzzard-659D8E62, B.Cu at (145.7, 94.6)
- added kibuzzard-659D8E71: G***, kibuzzard-659D8E71, B.Cu at (145.7, 95.9)
- added kibuzzard-659D9D0E: G***, kibuzzard-659D9D0E, F.Cu at (157.5, 92.1)
- added kibuzzard-659D9D29: G***, kibuzzard-659D9D29, F.Cu at (157.5, 101.0)
- added kibuzzard-659D9D38: G***, kibuzzard-659D9D38, F.Cu at (155.1, 97.9)
- added kibuzzard-659D9D4E: G***, kibuzzard-659D9D4E, F.Cu at (139.7, 91.9)
- added kibuzzard-659D9D68: G***, kibuzzard-659D9D68, F.Cu at (139.7, 101.0)
- added kibuzzard-659D9D77: G***, kibuzzard-659D9D77, F.Cu at (142.0, 96.5)
- C4: value C_Small -> 10pF
- R1, R2, R4, R5: value R_Small -> 10k
Routing:
- net GND: vias 6 -> 12
