File: KiCad/OPA990 Breakout.kicad_sch (KiCad schematic)
At the start: 13 parts, among them J1 Conn_01x03, J2 Conn_01x03, U1 OPA99X

Commit message: renamed files
Parts:
- removed D1: BAT54S, Package_TO_SOT_SMD:SOT-23, symbol friedElectronicsSymbols:BAT54S
- added C2: 10nF, Capacitor_SMD:C_0603_1608Metric, symbol Device:C_Small
- added D1: BAT54S, Package_TO_SOT_SMD:SOT-23-3, symbol Fried_Electronics_Symbols:BAT54S
- added R3: 100R, Resistor_SMD:R_0603_1608Metric, symbol Device:R_Small
- renumbered C2 to C3, C3 to C4, JP2 to JP1, JP1 to JP2, R3 to R4, R4 to R5
Connections:
- net GND: now also C2.2, D1.1 (A)
- net OUT: now also R3.2; no longer J2.2 (Pin_2)
- net VIO: now also D1.2 (K)
- new net: C2.1, D1.3 (COM), D1.3 (COM), J2.2 (Pin_2), R3.1
Other:
- title: Operational Amplifier Breakout -> OPA990 Breakout
- moved on the sheet: C1, C3, C4, J1, R1, R2, R4, R5, U1

Commit message: updated kicad files
Parts:
- removed U1: OPA99X, Package_TO_SOT_SMD:SOT-23-5, symbol friedElectronicsSymbols:OPA99X
- added U1: OPA99X, Package_TO_SOT_SMD:SOT-23-5, symbol Fried_Electronics_Symbols:OPA99X
- C1, C3: Manufacturer Part Number (none) -> 885012206095; Mouser Part Number (none) -> 710-885012206095
- C2: Manufacturer Part Number (none) -> CL10B103KB8NNNL; Mouser Part Number (none) -> 187-CL10B103KB8NNNL
- C4: value C_Small -> 10pF; Manufacturer Part Number (none) -> VJ0603A100GXACW1BC; Mouser Part Number (none) -> 77-VJ0603A100GXACBC
- D1: Manufacturer Part Number (none) -> BAT54S-7-F; Mouser Part Number (none) -> 621-BAT54S-F
- J1, J2: Manufacturer Part Number (none) -> 22-28-4030; Mouser Part Number (none) -> 538-22-28-4030
- JP1, JP2: now left out of the parts list
- R1, R2, R4, R5: value R_Small -> 10k; Manufacturer Part Number (none) -> RN73R1JTTD1002B25; Mouser Part Number (none) -> 660-RN73R1JTD1002B25
- R3: Manufacturer Part Number (none) -> RN73R1JTTD1000B25; Mouser Part Number (none) -> 660-RN73R1JTD1000B25
Connections:
- net IN+: now also U1.3 (+)
- net IN-: now also U1.4 (-)
- net OUT: now also U1.1
- net VDD: now also U1.5 (V+)
- net VSS: now also U1.2 (V-)
Other:
- moved on the sheet: C1, C2, C3, C4, D1A, D1B, J1, J2, JP1, JP2, R1, R2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
